Commit message: upload day2 progress

File: src/ntust_robot_description/urdf/urdf_test.urdf (robot description, URDF)
Before this commit: robot myfirst, 7 links, 6 joints
Links:
- link base_link: mass None -> 0.5
- link finger_left: mass None -> 0.05
- link finger_right: mass None -> 0.05
- link gripper_base: mass None -> 0.2
- link link1: mass None -> 0.4
- link link2: mass None -> 0.6
- link link3: mass None -> 0.6
